File: schema.sch (EAGLE design)
At the start: 21 parts, among them Q1 2N2907

Commit message: Version 2
Parts:
- removed C1: 2200uF, SparkFun-Capacitors:100UF-25V-20%(PTH)
- removed CH_PD, FLASH: OFF, adafruit:EG1218S
- removed D1: 1N4004, adafruit:1N4004
- removed FLOAT: 3.3v, pinhead:PINHD-1X2
- removed HUM_SENSOR: VCC_GND_D0_A0, pinhead:PINHD-1X4
- removed IN, MOTOR, TO_SENSOR: 5V, pinhead:PINHD-1X2
- removed IN+, IN-: 5v, pinhead:PINHD-1X1
- removed JACK: 5V IN, con-conrad:733989-5
- removed MDL1: ESP-12, ESP8266-ESP12E:ESP8266-12EESP8266-ESP12E
- removed OUT: 3.3V, pinhead:PINHD-1X2
- removed OUT+, OUT-: 3.3v, pinhead:PINHD-1X1
- removed Q1: 2N2907, adafruit:2N2907
- removed R1, R2: 300, adafruit:FLIPFLOP-RES
- removed WORKING_LED: 3.3v, adafruit:LED3MM
- added 5V: +5V, con-conrad:733989-5
- added BOOST_IN, SENSOR: (no value), pinhead:PINHD-1X3
- added BOOST_OUT, FLOAT_SW, PUMP: (no value), pinhead:PINHD-1X2
- added C2: 2200uF, SparkFun-Capacitors:100UF-25V-20%(PTH)
- added D2: 1N4148DO35-7, diode:1N4148DO35-7
- added FLASH_MODE, ON/OFF: TL36PO, switch:TL36PO
- added FLASH_UART: (no value), pinhead:PINHD-1X4
- added LED1: WORK, led:LED3MM
- added R4, R5, R6, R7: 10k, resistor:R-EU_0309/V
- added R8: 220, resistor:R-EU_0309/V
- added S1: RST_SW, switch-omron:10-XX
- added T1: 2N2222, transistor:2N2222
- added U1: ESP12E, esp8266modules:ESP12ESMD
- R3: device adafruit:FLIPFLOP-RES -> resistor:R-EU_0309/V
Connections:
- removed net N$1: HUM_SENSOR.4, IN.1
- removed net N$10: FLASH.P, MDL1.GPIO0
- removed net N$12: D1.C, MOTOR.1, Q1.C
- removed net N$13: FLOAT.1, MDL1.GPIO4, R3.1
- removed net N$2: MDL1.GPIO5, Q1.B
- removed net N$3: C1.+, CH_PD.P, FLOAT.2, MDL1.VCC, OUT+.1
- removed net N$4: CH_PD.S, MDL1.CH_PD
- removed net N$5: HUM_SENSOR.1, IN+.1, JACK.1, Q1.E
- removed net N$6: MDL1.ADC, OUT.1
- removed net N$7: MDL1.GPIO12, R1.2
- removed net N$8: R1.1, WORKING_LED.A
- removed net N$9: MDL1.GPIO15, R2.2
- new net +3V3: BOOST_OUT.2, C2.+, FLASH_UART.3, FLOAT_SW.1, ON/OFF.P, R7.1, SENSOR.2, U1.VCC
- new net +5V: 5V.1, BOOST_IN.1, BOOST_IN.3, D2.C, PUMP.1
- new net ADC: SENSOR.3, U1.ADC
- new net CH_PD: R6.1, U1.CH_PD
- new net CH_PD_S: ON/OFF.S, R6.2
- new net GPIO0: FLASH_MODE.S, U1.GPIO0
- new net GPIO12: R3.1, U1.GPIO12
- new net GPIO12D: LED1.A, R3.2
- new net GPIO15: R5.2, U1.GPIO15
- new net GPIO4: FLOAT_SW.2, R4.2, U1.GPIO4
- new net GPIO5: R8.1, U1.GPIO5
- new net GPIO5_T: R8.2, T1.B
- new net PUMP_GND: D2.A, PUMP.2, T1.E
- new net RST: S1.P1, U1.RESET
- new net RST_R: R7.2, S1.P
- new net RX: FLASH_UART.2, U1.RX
- new net TX: FLASH_UART.1, U1.TX
- net GND: now also 5V.2, 5V.3, BOOST_IN.2, BOOST_OUT.1, C2.-, FLASH_MODE.P, FLASH_UART.4, LED1.C, R4.1, R5.1, S1.S, S1.S1, SENSOR.1, T1.C, U1.GND; no longer C1.-, D1.A, FLASH.S, HUM_SENSOR.2, IN-.1, IN.2, JACK.2, JACK.3, MDL1.GND, MOTOR.2, OUT-.1, OUT.2, R2.1, R3.2, TO_SENSOR.1, WORKING_LED.C

Commit message: Circuit Update
Parts:
- removed ON/OFF: TL36PO, switch:TL36PO
- removed R8: 220, resistor:R-EU_0309/V
- removed SENSOR: (no value), pinhead:PINHD-1X3
- added JP1: MOISTURE, pinhead:PINHD-1X3
- added R1: 14k, pot:TRIM_EU-CA6V
- added R2: 10k, resistor:R-EU_0309/V
- added S2: RST_SW, switch-omron:10-XX
- JP2: value (none) -> BUCK_IN
- JP3: value (none) -> BUCK_OUT
- JP4: value (none) -> FLASH
- JP5: value (none) -> PUMP
- JP6: value (none) -> WATER_LOW
- R6: value 10k -> 220
- S1: value RST_SW -> TL36PO; device switch-omron:10-XX -> switch:TL36PO
- renumbered 5V to X1, BOOST_IN to JP2, BOOST_OUT to JP3, C2 to C1, D2 to D1, FLASH_MODE to S3, FLASH_UART to JP4, FLOAT_SW to JP6, PUMP to JP5
Connections:
- net +3V3: now also JP1.2, R4.1, S1.P; no longer ON/OFF.P, R7.1, SENSOR.2
- net ADC: now also JP1.3, R1.A; no longer SENSOR.3
- net CH_PD: now also R2.1; no longer R6.1
- net CH_PD_S: now also R2.2, S1.S; no longer ON/OFF.S, R6.2
- net GND: now also JP1.1, R1.S, R7.1, S2.S, S2.S1; no longer R4.1, S1.S, S1.S1, SENSOR.1
- net GPIO4: now also R7.2; no longer R4.2
- net GPIO5: now also R6.1; no longer R8.1
- net GPIO5_T: now also R6.2; no longer R8.2
- net RST: now also S2.P1; no longer S1.P1
- net RST_R: now also R4.2, S2.P; no longer R7.2, S1.P
Other:
- moved on the sheet: R4, R6, R7

Commit message: Changed Buck
Parts:
- removed JP2: BUCK_IN, pinhead:PINHD-1X3
- removed JP3: BUCK_OUT, pinhead:PINHD-1X2
- added U2: LM2596-L, hi-link:LM2596-L
Connections:
- net +3V3: now also U2.OUT+; no longer JP3.2
- net +5V: now also U2.IN+; no longer JP2.1, JP2.3
- net GND: now also U2.IN-, U2.OUT-; no longer JP2.2, JP3.1
Other:
- moved on the sheet: X1
Changed lines of the file:
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@@
 <part name="GND7" library="supply1" deviceset="GND" device=""/>
 <part name="X1" library="con-conrad" deviceset="73398?" device="9-5" value="+5V"/>
-<part name="JP2" library="pinhead" deviceset="PINHD-1X3" device="" value="BUCK_IN"/>
 <part name="P+1" library="supply1" deviceset="+5V" device=""/>
 <part name="GND1" library="supply1" deviceset="GND" device=""/>
-<part name="JP3" library="pinhead" deviceset="PINHD-1X2" device="" value="BUCK_OUT"/>
 <part name="GND5" library="supply1" deviceset="GND" device=""/>
 <part name="C1" library="SparkFun-Capacitors" deviceset="100UF-25V-20%(PTH)" device="" value="2200uF"/>
@@
 <part name="GND4" library="supply1" deviceset="GND" device=""/>
 <part name="R1" library="pot" deviceset="TRIM_EU-" device="CA6V" value="14k"/>
+<part name="U2" library="hi-link" deviceset="LM2596-L" device=""/>
 </parts>
 <sheets>
@@
 <instance part="+3V35" gate="G$1" x="-58.42" y="261.62" rot="R180"/>
 <instance part="GND7" gate="1" x="-55.88" y="259.08"/>
-<instance part="X1" gate="G$1" x="-154.94" y="203.2" rot="R180"/>
-<instance part="JP2" gate="A" x="-127" y="203.2"/>
-<instance part="P+1" gate="1" x="-144.78" y="195.58" rot="R180"/>
-<instance part="GND1" gate="1" x="-137.16" y="195.58"/>
-<instance part="JP3" gate="G$1" x="-114.3" y="205.74" rot="R180"/>
+<instance part="X1" gate="G$1" x="-154.94" y="205.74" rot="MR0"/>
+<instance part="P+1" gate="1" x="-144.78" y="213.36"/>
+<instance part="GND1" gate="1" x="-144.78" y="198.12"/>
 <instance part="GND5" gate="1" x="-104.14" y="200.66"/>
 <instance part="C1" gate="G$1" x="-86.36" y="218.44" rot="R90"/>
@@
 <instance part="GND4" gate="1" x="-114.3" y="274.32"/>
 <instance part="R1" gate="1" x="-119.38" y="279.4" rot="MR180"/>
+<instance part="U2" gate="G$1" x="-127" y="205.74"/>
 </instances>
 <busses>
@@
 </segment>
 <segment>
-<pinref part="X1" gate="G$1" pin="3"/>
-<pinref part="X1" gate="G$1" pin="2"/>
-<wire x1="-149.86" y1="203.2" x2="-149.86" y2="205.74" width="0.1524" layer="91"/>
-<pinref part="JP2" gate="A" pin="2"/>
-<wire x1="-149.86" y1="203.2" x2="-137.16" y2="203.2" width="0.1524" layer="91"/>
-<pinref part="GND1" gate="1" pin="GND"/>
-<wire x1="-137.16" y1="203.2" x2="-129.54" y2="203.2" width="0.1524" layer="91"/>
-<wire x1="-137.16" y1="198.12" x2="-137.16" y2="203.2" width="0.1524" layer="91"/>
-<junction x="-137.16" y="203.2"/>
-<junction x="-149.86" y="203.2"/>
-</segment>
-<segment>
-<pinref part="JP3" gate="G$1" pin="1"/>
 <pinref part="GND5" gate="1" pin="GND"/>
-<wire x1="-111.76" y1="203.2" x2="-104.14" y2="203.2" width="0.1524" layer="91"/>
 <pinref part="U1" gate="G$1" pin="GND"/>
 <pinref part="C1" gate="G$1" pin="-"/>
+<wire x1="-109.22" y1="203.2" x2="-104.14" y2="203.2" width="0.1524" layer="91"/>
 <wire x1="-68.58" y1="241.3" x2="-68.58" y2="218.44" width="0.1524" layer="91"/>
 <wire x1="-68.58" y1="218.44" x2="-81.28" y2="218.44" width="0.1524" layer="91"/>
@@
 <junction x="-81.28" y="218.44"/>
 <junction x="-104.14" y="203.2"/>
+<pinref part="U2" gate="G$1" pin="OUT-"/>
 </segment>
 <segment>
@@
 <wire x1="-114.3" y1="276.86" x2="-114.3" y2="279.4" width="0.1524" layer="91"/>
 </segment>
+<segment>
+<pinref part="X1" gate="G$1" pin="3"/>
+<pinref part="X1" gate="G$1" pin="2"/>
+<wire x1="-149.86" y1="205.74" x2="-149.86" y2="203.2" width="0.1524" layer="91"/>
+<pinref part="U2" gate="G$1" pin="IN-"/>
+<wire x1="-149.86" y1="203.2" x2="-144.78" y2="203.2" width="0.1524" layer="91"/>
+<junction x="-149.86" y="203.2"/>
+<pinref part="GND1" gate="1" pin="GND"/>
+<wire x1="-144.78" y1="203.2" x2="-142.24" y2="203.2" width="0.1524" layer="91"/>
+<wire x1="-144.78" y1="200.66" x2="-144.78" y2="203.2" width="0.1524" layer="91"/>
+<junction x="-144.78" y="203.2"/>
+</segment>
 </net>
 <net name="+3V3" class="0">
@@
 </segment>
 <segment>
-<pinref part="JP3" gate="G$1" pin="2"/>
-<wire x1="-111.76" y1="205.74" x2="-99.06" y2="205.74" width="0.1524" layer="91"/>
 <pinref part="U1" gate="G$1" pin="VCC"/>
 <pinref part="C1" gate="G$1" pin="+"/>
-<wire x1="-99.06" y1="205.74" x2="-88.9" y2="205.74" width="0.1524" layer="91"/>
+<wire x1="-99.06" y1="208.28" x2="-88.9" y2="208.28" width="0.1524" layer="91"/>
 <wire x1="-101.6" y1="241.3" x2="-101.6" y2="218.44" width="0.1524" layer="91"/>
 <wire x1="-101.6" y1="218.44" x2="-88.9" y2="218.44" width="0.1524" layer="91"/>
-<wire x1="-88.9" y1="218.44" x2="-88.9" y2="205.74" width="0.1524" layer="91"/>
+<wire x1="-88.9" y1="218.44" x2="-88.9" y2="208.28" width="0.1524" layer="91"/>
 <junction x="-88.9" y="218.44"/>
 <pinref part="+3V34" gate="G$1" pin="+3V3"/>
-<wire x1="-99.06" y1="200.66" x2="-99.06" y2="205.74" width="0.1524" layer="91"/>
-<junction x="-99.06" y="205.74"/>
+<wire x1="-99.06" y1="200.66" x2="-99.06" y2="208.28" width="0.1524" layer="91"/>
+<pinref part="U2" gate="G$1" pin="OUT+"/>
+<wire x1="-99.06" y1="208.28" x2="-109.22" y2="208.28" width="0.1524" layer="91"/>
+<junction x="-99.06" y="208.28"/>
 </segment>
 </net>
@@
 </net>
 <net name="+5V" class="0">
-<segment>
-<pinref part="X1" gate="G$1" pin="1"/>
-<wire x1="-149.86" y1="200.66" x2="-144.78" y2="200.66" width="0.1524" layer="91"/>
-<wire x1="-144.78" y1="200.66" x2="-144.78" y2="205.74" width="0.1524" layer="91"/>
-<pinref part="JP2" gate="A" pin="1"/>
-<wire x1="-129.54" y1="205.74" x2="-144.78" y2="205.74" width="0.1524" layer="91"/>
-<pinref part="JP2" gate="A" pin="3"/>
-<wire x1="-144.78" y1="200.66" x2="-129.54" y2="200.66" width="0.1524" layer="91"/>
-<pinref part="P+1" gate="1" pin="+5V"/>
-<wire x1="-144.78" y1="198.12" x2="-144.78" y2="200.66" width="0.1524" layer="91"/>
-<junction x="-144.78" y="200.66"/>
-</segment>
 <segment>
 <pinref part="D1" gate="G$1" pin="C"/>
@@
 <junction x="-35.56" y="203.2"/>
 </segment>
-</net>
+<segment>
+<pinref part="X1" gate="G$1" pin="1"/>
+<pinref part="U2" gate="G$1" pin="IN+"/>
+<wire x1="-149.86" y1="208.28" x2="-144.78" y2="208.28" width="0.1524" layer="91"/>
+<pinref part="P+1" gate="1" pin="+5V"/>
+<wire x1="-144.78" y1="208.28" x2="-142.24" y2="208.28" width="0.1524" layer="91"/>
+<wire x1="-144.78" y1="210.82" x2="-144.78" y2="208.28" width="0.1524" layer="91"/>
+<junction x="-144.78" y="208.28"/>
+</segment>
+</net>
